File: KiCad Designs/EGR101-Module/EGR 101.kicad_sch (KiCad schematic)
At the start: 15 parts, among them J1 RS485 Interface, J2 VEML7700-1, J3 VEML7700-2, U1 MAX3485, U2 LMR33630BDDA, U3 113991054

Commit message: Finished Module V1.1
Parts:
- added J4: NEO-6M, Connector_PinHeader_1.00mm:PinHeader_1x04_P1.00mm_Vertical, symbol Connector_Generic:Conn_01x04
- added R4, R5, R6, R8: 4.7 kΩ, Capacitor_SMD:C_0402_1005Metric_Pad0.74x0.62mm_HandSolder, symbol Device:R
- J1: value RS485 Interface -> GX12
Connections:
- net at C4.1, C5.1, J2.1 (Pin_1)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: now also J4.1 (Pin_1), R4.2, R5.2, R6.2, R8.2
- net at C1.2, C2.2, C4.2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: now also J4.4 (Pin_4)
- net at J3.4 (Pin_4), U3.2 (D1): now also R4.1
- net at J3.5 (Pin_5), U3.1 (D0): now also R8.1
- net at J2.4 (Pin_4), U3.6 (D5): now also R6.1
- net at J2.5 (Pin_5), U3.5 (D4): now also R5.1
- net at U3.10 (D9): now also J4.3 (Pin_3)
- net at U3.9 (D8): now also J4.2 (Pin_2)
- no-connect marks 11 -> 9
Other:
- note added: "I2C Pull-up Resistors"
- title: (none) -> EGR101 Module Schematic
- moved on the sheet: C1, C2, C3, C4, C5, J1, J2, J3, L1, R1, R2, R3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

Commit message: More udaptes
Parts:
- added J5: Switch, Connector_PinHeader_2.54mm:PinHeader_1x02_P2.54mm_Vertical, symbol Connector_Generic:Conn_01x02
- J1, J4: footprint Connector_PinHeader_1.00mm:PinHeader_1x04_P1.00mm_Vertical -> Connector_PinHeader_2.54mm:PinHeader_1x04_P2.54mm_Vertical
- J2, J3: footprint Connector_PinHeader_1.00mm:PinHeader_1x05_P1.00mm_Vertical -> Connector_PinHeader_2.54mm:PinHeader_1x05_P2.54mm_Vertical
Connections:
- net at C1.2, C2.2, C4.2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: now also J5.2 (Pin_2)
- net at U3.11 (D10): now also J5.1 (Pin_1)
- no-connect marks 9 -> 8
Changed lines of the file:
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@@
+	)
+	(junction
+		(at 177.8 100.33)
+		(diameter 0)
+		(color 0 0 0 0)
 	)
 	(junction
@@
 	)
 	(no_connect
-		(at 166.37 101.6)
-	)
-	(no_connect
 		(at 166.37 93.98)
 	)
@@
 	(wire
 		(pts
+			(xy 175.26 101.6) (xy 166.37 101.6)
+		)
+		(stroke
+			(width 0)
+			(type default)
+		)
+	)
+	(wire
+		(pts
 			(xy 102.87 62.23) (xy 102.87 63.5)
 		)
@@
 	(wire
 		(pts
+			(xy 177.8 100.33) (xy 177.8 109.22)
+		)
+		(stroke
+			(width 0)
+			(type default)
+		)
+	)
+	(wire
+		(pts
 			(xy 189.23 72.39) (xy 189.23 74.93)
 		)
@@
 	(wire
 		(pts
-			(xy 177.8 91.44) (xy 177.8 109.22)
+			(xy 175.26 97.79) (xy 175.26 101.6)
+		)
+		(stroke
+			(width 0)
+			(type default)
+		)
+	)
+	(wire
+		(pts
+			(xy 177.8 91.44) (xy 177.8 100.33)
 		)
 		(stroke
@@
 	(wire
 		(pts
+			(xy 195.58 97.79) (xy 175.26 97.79)
+		)
+		(stroke
+			(width 0)
+			(type default)
+		)
+	)
+	(wire
+		(pts
 			(xy 153.67 55.88) (xy 154.94 55.88)
+		)
+		(stroke
+			(width 0)
+			(type default)
+		)
+	)
+	(wire
+		(pts
+			(xy 177.8 100.33) (xy 195.58 100.33)
 		)
 		(stroke
@@
 			)
 		)
-		(property "Footprint" "Connector_PinHeader_1.00mm:PinHeader_1x05_P1.00mm_Vertical"
+		(property "Footprint" "Connector_PinHeader_2.54mm:PinHeader_1x05_P2.54mm_Vertical"
 			(at 200.66 72.39 0)
 			(effects
@@
 			)
 		)
-		(property "Footprint" "Connector_PinHeader_1.00mm:PinHeader_1x04_P1.00mm_Vertical"
+		(property "Footprint" "Connector_PinHeader_2.54mm:PinHeader_1x04_P2.54mm_Vertical"
 			(at 73.66 60.96 0)
 			(effects
@@
 			)
 		)
-		(property "Footprint" "Connector_PinHeader_1.00mm:PinHeader_1x04_P1.00mm_Vertical"
+		(property "Footprint" "Connector_PinHeader_2.54mm:PinHeader_1x04_P2.54mm_Vertical"
 			(at 200.66 86.36 0)
 			(effects
@@
 			)
 		)
-		(property "Footprint" "Connector_PinHeader_1.00mm:PinHeader_1x05_P1.00mm_Vertical"
+		(property "Footprint" "Connector_PinHeader_2.54mm:PinHeader_1x05_P2.54mm_Vertical"
 			(at 200.66 55.88 0)
 			(effects
@@
 					(unit 1)
 				)
+			)
+		)
+	)
+	(symbol
+		(lib_id "Connector_Generic:Conn_01x02")
+		(at 200.66 97.79 0)
+		(unit 1)
+		(exclude_from_sim no)
+		(in_bom yes)
+		(on_board yes)
+		(dnp no)
+		(fields_autoplaced yes)
+		(property "Reference" "J5"
+			(at 203.2 97.7899 0)
+			(effects
+				(font
+					(size 1.27 1.27)
+				)
+				(justify left)
+			)
+		)
+		(property "Value" "Switch"
+			(at 203.2 100.3299 0)
+			(effects
+				(font
+					(size 1.27 1.27)
+				)
+				(justify left)
+			)
+		)
+		(property "Footprint" "Connector_PinHeader_2.54mm:PinHeader_1x02_P2.54mm_Vertical"
+			(at 200.66 97.79 0)
+			(effects
+				(font
+					(size 1.27 1.27)
+				)
+				(hide yes)
+			)
+		)
+		(property "Datasheet" "~"
+			(at 200.66 97.79 0)
+			(effects
+				(font
+					(size 1.27 1.27)
+				)
+				(hide yes)
+			)
+		)
+		(property "Description" "Generic connector, single row, 01x02, script generated (kicad-library-utils/schlib/autogen/connector/)"
+			(at 200.66 97.79 0)
+			(effects
+				(font
+					(size 1.27 1.27)
+				)
+				(hide yes)
+			)
+		)
+		(pin "2"
+		)
+		(pin "1"
+		)
+		(instances
+			(project ""
+				(path "/24fc8130-f04e-4e0f-be15-fcd1c3e02d49"
+					(reference "J5")
+					(unit 1)
+				)

Commit message: Module V1.0 Done
Parts:
- removed C2: 220 nF, Capacitor_SMD:C_0402_1005Metric_Pad0.74x0.62mm_HandSolder, symbol Device:C_Small
- removed R1: 43.2 kΩ, Resistor_SMD:R_0402_1005Metric_Pad0.72x0.64mm_HandSolder, symbol Device:R
- removed R2: 100 kΩ, Resistor_SMD:R_0402_1005Metric_Pad0.72x0.64mm_HandSolder, symbol Device:R
- removed U2: LMR33630BDDA, Package_SO:Texas_HSOP-8-1EP_3.9x4.9mm_P1.27mm_ThermalVias, symbol Regulator_Switching:LMR33630BDDA
- added H1, H2, H3, H4: MountingHole, MountingHole:MountingHole_2.7mm, symbol Mechanical:MountingHole
- added U2: AP63203WU, Package_TO_SOT_SMD:TSOT-23-6, symbol Regulator_Switching:AP63205WU
- C3: value 0.1 uF -> 100 nF
- J1: value GX12 -> External Connection
- L1: value 2.2 uH -> 3.9 uH
Connections:
- net at C4.1, C5.1, J2.1 (Pin_1)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: now also U2.1 (FB)
- net at L1.1: now also C3.2, U2.5 (SW); no longer C3.1
- net at C1.1, J1.4 (Pin_4): now also U2.2 (EN), U2.3 (IN)
- net at C1.2, C4.2, C5.2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: now also U2.4 (GND)
- net at R3.1, U1.6 (A): now also J1.2 (Pin_2); no longer J1.1 (Pin_1)
- net at R3.2, U1.7 (B): now also J1.1 (Pin_1); no longer J1.2 (Pin_2)
- new net: C3.1, U2.6 (BST)
- no-connect marks 8 -> 7
Other:
- note added: "MAX3485"
- moved on the sheet: C1, C3, C4, C5, J1, J2, J3, J4, J5, L1, R3, U1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

Commit message: Chamber PCB Finished
Other:
- company: (none) -> Duke University - EGR 101
- title: EGR101 Module Schematic -> ORCA Module Board - V1.0
- moved on the sheet: C1, C3, C4, C5, H1, H2, H3, H4, J1, J2, J3, J4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

Commit message: Module & Chamber V1.0 PCB Complete
Parts:
- C4, C5: footprint Capacitor_SMD:C_0201_0603Metric_Pad0.64x0.40mm_HandSolder -> Capacitor_SMD:C_0603_1608Metric_Pad1.08x0.95mm_HandSolder
Changed lines of the file:
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@@
 			)
 		)
-		(property "Footprint" "Capacitor_SMD:C_0201_0603Metric_Pad0.64x0.40mm_HandSolder"
+		(property "Footprint" "Capacitor_SMD:C_0603_1608Metric_Pad1.08x0.95mm_HandSolder"
 			(at 177.8 63.5 0)
 			(effects
@@
 			)
 		)
-		(property "Footprint" "Capacitor_SMD:C_0201_0603Metric_Pad0.64x0.40mm_HandSolder"
+		(property "Footprint" "Capacitor_SMD:C_0603_1608Metric_Pad1.08x0.95mm_HandSolder"
 			(at 189.23 63.5 0)
 			(effects
